Commit message: navigation of custom urdf done

File: src/autobot/urdf/lidar.xacro (robot description, xacro)
@@ -1,5 +1,5 @@
 <?xml version="1.0"?>
 <robot xmlns:xacro="http://www.ros.org/wiki/xacro" >
-    <joint name="laser_joint" type="fixed">
+    <!-- <joint name="laser_joint" type="fixed">
         <parent link="chassis"/>
         <child link="laser_frame"/>
@@ -28,10 +28,63 @@
             <origin xyz="0 0 0" rpy="0 0 0"/>
         </xacro:inertial_cylinder>
-    </link>
-    <gazebo reference="laser_frame">
+    </link> -->
+    <link
+    name="lidar">
+    <inertial>
+      <origin
+        xyz="-0.002361 -1.4968E-05 0.019299"
+        rpy="0 0 0" />
+      <mass
+        value="0.16538" />
+      <inertia
+        ixx="7.8866E-05"
+        ixy="4.8738E-08"
+        ixz="2.1848E-06"
+        iyy="7.519E-05"
+        iyz="2.8958E-08"
+        izz="0.00010995" />
+    </inertial>
+    <visual>
+      <origin
+        xyz="0 0 0"
+        rpy="0 0 0" />
+      <geometry>
+        <mesh
+          filename="package://autobot/meshes/lidar.STL" />
+      </geometry>
+      <material
+        name="">
+        <color
+          rgba="0.75294 0.75294 0.75294 0.4" />
+      </material>
+    </visual>
+    <collision>
+      <origin
+        xyz="0 0 0"
+        rpy="0 0 0" />
+      <geometry>
+        <mesh
+          filename="package://autobot/meshes/lidar.STL" />
+      </geometry>
+    </collision>
+  </link>
+  <joint
+    name="lidar_joint"
+    type="fixed">
+    <origin
+      xyz="0.063868 0.006608 0.050657"
+      rpy="0 0 0" />
+    <parent
+      link="base_link" />
+    <child
+      link="lidar" />
+    <axis
+      xyz="0 0 0" />
+  </joint>
+    <gazebo reference="lidar">
         <material>Gazebo/Black</material>
         <sensor name="laser" type="ray">
             <pose> 0 0 0 0 0 0 </pose>
-            <visualize>false</visualize>
+            <visualize>true</visualize>
             <update_rate>10</update_rate>
             <ray>
@@ -53,5 +106,5 @@
                 </ros>
                 <output_type>sensor_msgs/LaserScan</output_type>
-                <frame_name>laser_frame</frame_name>
+                <frame_name>lidar</frame_name>
             </plugin>
         </sensor>

File: src/autobot/urdf/robot.urdf.xacro (robot description, xacro)
@@ -10,5 +10,5 @@
         <xacro:include filename="gazebo_control.xacro" />
     </xacro:unless>
-    <!-- <xacro:include filename="lidar.xacro" /> -->
+    <xacro:include filename="lidar.xacro" />
     <!-- <xacro:include filename="camera.xacro" /> -->
     <!-- <xacro:include filename="depth_camera.xacro" /> -->

File: src/autobot/urdf/robot_core.xacro (robot description, xacro)
@@ -108,5 +108,5 @@
     <inertial>
         <origin xyz="5.5511E-17 7.6762E-16 4.1633E-17" rpy="0 0 0" />
-        <mass value="0.3" />
+        <mass value="0.4" />
         <inertia ixx="9.1441E-05" ixy="1.239E-18" ixz="3.9667E-21" iyy="0.00018051" iyz="-1.6989E-19" izz="9.1441E-05" />
     </inertial>
@@ -141,57 +141,4 @@
     </gazebo>
 </joint>
-  <link
-    name="lidar">
-    <inertial>
-      <origin
-        xyz="-0.002361 -1.4968E-05 0.019299"
-        rpy="0 0 0" />
-      <mass
-        value="0.16538" />
-      <inertia
-        ixx="7.8866E-05"
-        ixy="4.8738E-08"
-        ixz="2.1848E-06"
-        iyy="7.519E-05"
-        iyz="2.8958E-08"
-        izz="0.00010995" />
-    </inertial>
-    <visual>
-      <origin
-        xyz="0 0 0"
-        rpy="0 0 0" />
-      <geometry>
-        <mesh
-          filename="package://autobot/meshes/lidar.STL" />
-      </geometry>
-      <material
-        name="">
-        <color
-          rgba="0.75294 0.75294 0.75294 0.4" />
-      </material>
-    </visual>
-    <collision>
-      <origin
-        xyz="0 0 0"
-        rpy="0 0 0" />
-      <geometry>
-        <mesh
-          filename="package://autobot/meshes/lidar.STL" />
-      </geometry>
-    </collision>
-  </link>
-  <joint
-    name="lidar_joint"
-    type="fixed">
-    <origin
-      xyz="0.063868 0.006608 0.050657"
-      rpy="0 0 0" />
-    <parent
-      link="base_link" />
-    <child
-      link="lidar" />
-    <axis
-      xyz="0 0 0" />
-  </joint>
   <link
     name="camera">
